File: hw/EEW-display.kicad_sch (KiCad schematic)
At the start: 47 parts, among them J1 USB4105-GF-A, J2 B2B-PH-K-S, Q1 SSM3J332R, SW1 PAGE/BOOT, SW2 ZOOM-IN, SW3 MODE, SW4 ZOOM-OUT, SW5 SLIDE_SW, U1 ESP32-S3-WROOM-1-N16R8, U2 MCP73831T-2ATI/OT, U3 SPX3819M5-L, U4 MAX98357A, U5 ILI9488 MCU I8080 8/16BIT 3/4, Y1 32.7680KHz

Commit message: Fixed Display Footprint and C1 capacitor value
Parts:
- C1: value 0.1uF -> 1uF; footprint Capacitor_SMD:C_0603_1608Metric -> Capacitor_SMD:C_0805_2012Metric; digikey 311-1344-1-ND -> 1276-1026-1-ND; distributor https://www.digikey.com/en/products/detail/yageo/CC0603ZRY5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 -> https://www.digikey.com/en/products/detail/yageo/CC0805ZRY5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
